Commit message: wip

File: urdf/omnitrak_sensores_URDF.xacro (robot description, xacro)
@@ -24,4 +24,8 @@
   </collision>
 </link>
+<link name="camera_link">
+</link>
+<link name="front_track_cam">
+</link>
 <link name="perfil_lateral_derecho_1">
   <inertial>
@@ -2337,4 +2341,9 @@
   <child link="d435_1"/>
 </joint>
+<joint name="d435i_fix" type="fixed">
+  <origin xyz="-0.000 0.0 -0.0" rpy="0 0 0"/>
+  <parent link="d435_1"/>
+  <child link="camera_link"/>
+</joint>
 <joint name="fixed_lidar1" type="fixed">
   <origin xyz="-0.01337 0.540008 -0.256719" rpy="0 0 0"/>
@@ -2352,4 +2361,9 @@
   <child link="td65_body_1"/>
 </joint>
+<joint name="t265_to_td65_fix" type="fixed">
+  <origin xyz="0.000 0.000 0.00" rpy="0 0 0"/>
+  <parent link="td65_body_1"/>
+  <child link="front_track_cam"/>
+</joint>
 <joint name="fixed_t265" type="fixed">
   <origin xyz="0.0365 0.409448 0.360978" rpy="0 0 0"/>
